File: pcbs/rpi-hat/main.sch (EAGLE design)
At the start: 18 parts, among them IC1 MCP23017SP2, U1 MCP3002-I/P

Commit message: chg
Parts:
- removed GENERAL_LED: RGBLED_CA-5MM, adafruit:RGBLED_CA-5MM
- removed JP2: (no value), adafruit:PINHD-1X12-CB
- removed R1, R2, R3: 47, adafruit:R-US_0204/7
- removed R4: (no value), pot:3RP/1610N
- added GRN, RED, YEL: (no value), adafruit:LED3MM
- added IC2: L293D, st-microelectronics:L293D
- added J1: (no value), SparkFun-Connectors:M07
- added J2, J3: 1X2-3.5MM, adafruit:1X2-3.5MM
Connections:
- net N$11 renamed MGPB0
- net N$13 renamed MGPB1
- net N$14 renamed MGPB2
- net N$15 renamed MGPB3
- net N$16 renamed MGPB4
- net N$17 renamed MGPB5
- removed net BAR_3: IC1.GPA2, JP2.6
- removed net BAR_4: IC1.GPA3, JP2.8
- removed net BAR_5: IC1.GPA4, JP2.10
- removed net BAR_6: IC1.GPA5, JP2.12
- removed net BAR_R: IC1.GPA1, JP2.4
- removed net BAR_T: IC1.GPA0, JP2.2
- removed net GBLUE: PCB1.GPIO21, R8.1
- removed net GGRN: PCB1.GPIO20, R7.1
- removed net GRED: PCB1.GPIO16, R6.1
- removed net N$10: JP2.11, JP2.9, R3.1
- removed net N$12: R4.A, R5.1
- removed net N$9: JP2.5, JP2.7, R2.1
- removed net POT: DISPLAY.3, R4.S
- new net +12V: IC2.VCC2, J2.1
- new net GPIO13: PCB1.GPIO13, R8.1
- new net GPIO22: IC2.2A, PCB1.GPIO22
- new net GPIO27: IC2.1A, PCB1.GPIO27
- new net GPIO5: PCB1.GPIO5, R6.1
- new net GPIO6: PCB1.GPIO6, R7.1
- new net N$1: IC1.GPA5, J1.7
- new net N$2: IC1.GPA4, J1.6
- new net N$3: IC1.GPA3, J1.5
- new net N$4: IC1.GPA2, J1.4
- new net N$5: IC1.GPA1, J1.3
- new net N$7: IC1.GPA0, J1.2
- new net OUT1: IC2.1Y, J3.1
- new net OUT2: IC2.2Y, J3.2
- new net PWM1: IC2.1-2EN, PCB1.GPIO17
- net 5V: now also IC2.VCC1
- net GND: now also GRN.C, IC2.GND1, IC2.GND2, J1.1, J2.2, RED.C, YEL.C; no longer GENERAL_LED.VCC, R1.2, R2.2, R3.2, R4.E
- net N$18: now also GRN.A; no longer GENERAL_LED.RED
- net N$19: now also YEL.A; no longer GENERAL_LED.GREEN
- net N$20: now also RED.A; no longer GENERAL_LED.BLUE
- net N$8: now also DISPLAY.3, R5.1; no longer JP2.1, JP2.3, R1.1
Other:
- moved on the sheet: DISPLAY, R5, R6, R7, R8

Commit message: fuck
Parts:
- IC1: value MCP23017SP2 -> MCP23017
- U1: value MCP3002-I/P -> MCP3002
Changed lines of the file:
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@@
 <part name="JP1" library="adafruit" deviceset="PINHD-1X3" device=""/>
 <part name="GND4" library="supply1" deviceset="GND" device=""/>
-<part name="U1" library="mcp" deviceset="MCP3002-I/P" device=""/>
+<part name="U1" library="mcp" deviceset="MCP3002-I/P" device="" value="MCP3002"/>
 <part name="P+4" library="supply1" deviceset="VCC" device=""/>
-<part name="IC1" library="adafruit" deviceset="MCP23017" device="SP2"/>
+<part name="IC1" library="adafruit" deviceset="MCP23017" device="SP2" value="MCP23017"/>
 <part name="GND3" library="supply1" deviceset="GND" device=""/>
 <part name="GND5" library="supply1" deviceset="GND" device=""/>

Commit message: board changes
Parts:
- removed R5: 1k, adafruit:R-US_0204/7
Connections:
- removed net N$8: DISPLAY.3, R5.1
- net GND: now also DISPLAY.3
- net VCC: no longer R5.2
Changed lines of the file:
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@@
 <part name="P+3" library="supply1" deviceset="VCC" device=""/>
 <part name="DISPLAY" library="con-lstb" deviceset="MA07-2" device=""/>
-<part name="R5" library="adafruit" deviceset="R-US_" device="0204/7" value="1k"/>
-<part name="P+5" library="supply1" deviceset="VCC" device=""/>
 <part name="GND11" library="supply1" deviceset="GND" device=""/>
 <part name="R6" library="adafruit" deviceset="R-US_" device="0204/7" value="270"/>
@@
 <part name="GND9" library="supply1" deviceset="GND" device=""/>
 <part name="GND10" library="supply1" deviceset="GND" device=""/>
-<part name="GND12" library="supply1" deviceset="GND" device=""/>
-<part name="GND15" library="supply1" deviceset="GND" device=""/>
+<part name="GND16" library="supply1" deviceset="GND" device=""/>
 </parts>
 <sheets>
@@
 <instance part="P+3" gate="VCC" x="266.7" y="5.08" rot="R90"/>
 <instance part="DISPLAY" gate="G$1" x="347.98" y="-33.02" rot="R180"/>
-<instance part="R5" gate="G$1" x="330.2" y="-27.94" rot="R180"/>
-<instance part="P+5" gate="VCC" x="322.58" y="-27.94" rot="R90"/>
 <instance part="GND11" gate="1" x="104.14" y="137.16" rot="R180"/>
 <instance part="R6" gate="G$1" x="81.28" y="63.5" rot="R270"/>
@@
 <instance part="GND9" gate="1" x="78.74" y="-33.02" rot="R270"/>
 <instance part="GND10" gate="1" x="78.74" y="-38.1" rot="R270"/>
-<instance part="GND12" gate="1" x="337.82" y="-25.4" rot="R270"/>
-<instance part="GND15" gate="1" x="337.82" y="-30.48" rot="R270"/>
+<instance part="GND16" gate="1" x="335.28" y="-27.94" rot="R270"/>
 </instances>
 <busses>
@@
 <segment>
 <pinref part="DISPLAY" gate="G$1" pin="1"/>
-<pinref part="GND12" gate="1" pin="GND"/>
-</segment>
-<segment>
+<pinref part="GND16" gate="1" pin="GND"/>
+<wire x1="340.36" y1="-25.4" x2="337.82" y2="-25.4" width="0.1524" layer="91"/>
+<wire x1="337.82" y1="-25.4" x2="337.82" y2="-27.94" width="0.1524" layer="91"/>
+<pinref part="DISPLAY" gate="G$1" pin="3"/>
+<wire x1="340.36" y1="-27.94" x2="337.82" y2="-27.94" width="0.1524" layer="91"/>
+<junction x="337.82" y="-27.94"/>
 <pinref part="DISPLAY" gate="G$1" pin="5"/>
-<pinref part="GND15" gate="1" pin="GND"/>
+<wire x1="340.36" y1="-30.48" x2="337.82" y2="-30.48" width="0.1524" layer="91"/>
+<wire x1="337.82" y1="-30.48" x2="337.82" y2="-27.94" width="0.1524" layer="91"/>
 </segment>
 </net>
@@
 <pinref part="IC1" gate="G$1" pin="!RESET"/>
 <pinref part="P+3" gate="VCC" pin="VCC"/>
-</segment>
-<segment>
-<pinref part="R5" gate="G$1" pin="2"/>
-<pinref part="P+5" gate="VCC" pin="VCC"/>
 </segment>
 <segment>
@@
 </segment>
 </net>
-<net name="N$8" class="0">
-<segment>
-<pinref part="R5" gate="G$1" pin="1"/>
-<pinref part="DISPLAY" gate="G$1" pin="3"/>
-<wire x1="335.28" y1="-27.94" x2="340.36" y2="-27.94" width="0.1524" layer="91"/>
-</segment>
-</net>
