File: pcbs/rpi-hat/main.brd (EAGLE design)
At the start: 85.1 x 55.9 mm, 18 parts, among them IC1 MCP23017SP2, U1 MCP3002-I/P

Commit message: chg
Parts:
- removed GENERAL_LED: RGBLED_CA-5MM, adafruit:LED5MMRGB
- removed JP2: (no value), adafruit:1X12-CB
- removed R1, R2, R3: 47, adafruit:0204/7
- removed R4: (no value), pot:3RP/1610N
- added GRN, RED, YEL: (no value), adafruit:LED3MM
- added IC2: L293D, st-microelectronics:DIL16
- added J1: (no value), SparkFun-Connectors:1X07
- added J2, J3: 1X2-3.5MM, adafruit:1X2-3.5MM
- moved JP1 68.7 mm to (15.2, 2.54)
- moved U1 48.6 mm to (33.0, 2.54), turned to 0 degrees
- moved DISPLAY 45.5 mm to (61.0, 31.8), turned to 270 degrees
- moved R5 42.2 mm to (55.9, 33.0)
- moved IC1 32.2 mm to (72.4, 20.3), turned to 270 degrees
- moved TSL2561 18.9 mm to (10.2, 44.5), turned to 0 degrees
- moved R6 15.5 mm to (63.5, 43.2)
- moved R7 13.1 mm to (69.8, 45.7)
- moved PCB1 5.39 mm to (0.00, 0.00)
- moved R8 3.81 mm to (76.2, 43.2)
- moved DHT22 2.84 mm to (45.7, 10.2)
- moved R9 1.80 mm to (49.5, 15.2)
Connections:
- net N$11 renamed MGPB0
- net N$13 renamed MGPB1
- net N$14 renamed MGPB2
- net N$15 renamed MGPB3
- net N$16 renamed MGPB4
- net N$17 renamed MGPB5
- removed net BAR_3: IC1.23, JP2.6
- removed net BAR_4: IC1.24, JP2.8
- removed net BAR_5: IC1.25, JP2.10
- removed net BAR_6: IC1.26, JP2.12
- removed net BAR_R: IC1.22, JP2.4
- removed net BAR_T: IC1.21, JP2.2
- removed net GBLUE: PCB1.P$40, R8.1
- removed net GGRN: PCB1.P$38, R7.1
- removed net GRED: PCB1.P$36, R6.1
- removed net N$10: JP2.11, JP2.9, R3.1
- removed net N$12: R4.1, R5.1
- removed net N$9: JP2.5, JP2.7, R2.1
- removed net POT: DISPLAY.3, R4.2
- new net +12V: IC2.8, J2.1
- new net GND3: IC2.13
- new net GND4: IC2.12
- new net GPIO13: PCB1.P$33, R8.1
- new net GPIO22: IC2.7, PCB1.P$15
- new net GPIO27: IC2.2, PCB1.P$13
- new net GPIO5: PCB1.P$29, R6.1
- new net GPIO6: PCB1.P$31, R7.1
- new net N$1: IC1.26, J1.7
- new net N$2: IC1.25, J1.6
- new net N$3: IC1.24, J1.5
- new net N$4: IC1.23, J1.4
- new net N$5: IC1.22, J1.3
- new net N$7: IC1.21, J1.2
- new net OUT1: IC2.3, J3.1
- new net OUT2: IC2.6, J3.2
- new net PWM1: IC2.1, PCB1.P$11
- net 5V: now also IC2.16
- net GND: now also GRN.K, IC2.4, IC2.5, J1.1, J2.2, RED.K, YEL.K; no longer GENERAL_LED.2, R1.2, R2.2, R3.2, R4.3
- net N$18: now also GRN.A; no longer GENERAL_LED.1
- net N$19: now also YEL.A; no longer GENERAL_LED.3
- net N$20: now also RED.A; no longer GENERAL_LED.4
- net N$8: now also DISPLAY.3, R5.1; no longer JP2.1, JP2.3, R1.1
Routing:
- net VCC: track 138.2 -> 0.00 mm
- net 5V: track 52.4 -> 148.8 mm
- net BAR_6: track 67.1 -> 0.00 mm
- net BAR_5: track 60.9 -> 0.00 mm
- net BAR_4: track 54.8 -> 0.00 mm
- net BAR_T: track 52.3 -> 0.00 mm
- net BAR_R: track 52.3 -> 0.00 mm
- net BAR_3: track 52.3 -> 0.00 mm
- net GPIO22: track 0.00 -> 47.3 mm
- net CE0: track 87.1 -> 48.6 mm, vias 0 -> 2
- net GPIO4: track 106.1 -> 69.6 mm, vias 1 -> 0
- net GPIO13: track 0.00 -> 32.2 mm
- net GPIO27: track 0.00 -> 31.3 mm
- net MOSI: track 78.4 -> 49.4 mm
- net PWM1: track 0.00 -> 27.7 mm
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- added copper zone on layer 1, net VCC
- removed copper zone on layer 1, net GND
Other:
- board text added: "+12V"
- board text added: "OUT1"
- board text added: "OUT2"
- board text added: "SCL"
- board text removed: "MOISTURE"
- board text removed: "MOISTURE LED BAR"

Commit message: fuck
Parts:
- IC1: value MCP23017SP2 -> MCP23017
- U1: value MCP3002-I/P -> MCP3002
Routing:
- net GPIO22: track 47.3 -> 71.4 mm
- net GPIO27: track 31.3 -> 54.0 mm
- net PWM1: track 27.7 -> 46.8 mm
Other:
- board text added: ""Nothing is work unless you'd rather be doing something else" - George Halas"
- board text added: "2017 Bilal Mahmoud"

Commit message: board changes
Parts:
- removed R5: 1k, adafruit:0204/7
Connections:
- removed net N$8: DISPLAY.3, R5.1
- net GND: now also DISPLAY.3
- net VCC: no longer R5.2
Routing:
- net N$8: track 3.81 -> 0.00 mm
Changed lines of the file:
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@@
 </element>
 <element name="PCB1" library="e14_Rpi2_RevA" package="RPI2" value="RPI2" x="0" y="0"/>
-<element name="R5" library="adafruit" package="0204/7" value="1k" x="55.88" y="33.02" smashed="yes" rot="R270">
-<attribute name="NAME" x="54.5846" y="30.48" size="0.9906" layer="21" ratio="12" rot="R90"/>
-<attribute name="VALUE" x="55.3974" y="34.6456" size="0.8128" layer="21" ratio="12" rot="R270"/>
-</element>
 <element name="R6" library="adafruit" package="0204/7" value="270" x="63.5" y="43.18" smashed="yes">
 <attribute name="NAME" x="64.77" y="40.6654" size="0.9906" layer="21" ratio="12"/>
@@
 </polygon>
 <contactref element="DISPLAY" pad="1"/>
+<contactref element="DISPLAY" pad="3"/>
 <contactref element="DISPLAY" pad="5"/>
+<wire x1="73.66" y1="50.8" x2="80.01" y2="50.8" width="0" layer="19" extent="1-1"/>
+<wire x1="67.31" y1="50.8" x2="73.66" y2="50.8" width="0" layer="19" extent="1-1"/>
+<wire x1="59.69" y1="39.37" x2="67.31" y2="50.8" width="0" layer="19" extent="1-1"/>
+<wire x1="59.69" y1="36.83" x2="59.69" y2="39.37" width="0" layer="19" extent="1-1"/>
+<wire x1="59.69" y1="34.29" x2="59.69" y2="36.83" width="0" layer="19" extent="1-1"/>
+<wire x1="68.58" y1="13.97" x2="59.69" y2="34.29" width="0" layer="19" extent="1-1"/>
+<wire x1="76.2" y1="8.89" x2="68.58" y2="13.97" width="0" layer="19" extent="1-1"/>
+<wire x1="76.2" y1="6.35" x2="76.2" y2="8.89" width="0" layer="19" extent="1-1"/>
+<wire x1="76.2" y1="3.81" x2="76.2" y2="6.35" width="0" layer="19" extent="1-1"/>
+<wire x1="82.55" y1="16.51" x2="76.2" y2="8.89" width="0" layer="19" extent="1-1"/>
+<wire x1="53.34" y1="10.16" x2="68.58" y2="13.97" width="0" layer="19" extent="1-1"/>
+<wire x1="25.4" y1="2.54" x2="53.34" y2="10.16" width="0" layer="19" extent="1-1"/>
+<wire x1="15.24" y1="2.54" x2="25.4" y2="2.54" width="0" layer="19" extent="1-1"/>
+<wire x1="5.08" y1="15.67" x2="15.24" y2="2.54" width="0" layer="19" extent="1-1"/>
+<wire x1="12.7" y1="19.05" x2="5.08" y2="15.67" width="0" layer="19" extent="1-1"/>
+<wire x1="12.7" y1="21.59" x2="12.7" y2="19.05" width="0" layer="19" extent="1-1"/>
+<wire x1="12.7" y1="44.45" x2="12.7" y2="21.59" width="0" layer="19" extent="1-1"/>
+<wire x1="18.5166" y1="51.2318" x2="12.7" y2="44.45" width="0" layer="19" extent="1-1"/>
 </signal>
 <signal name="VCC">
@@
 <contactref element="IC1" pad="9"/>
 <contactref element="IC1" pad="18"/>
-<contactref element="R5" pad="2"/>
 <contactref element="DHT22" pad="1"/>
 <contactref element="R9" pad="2"/>
@@
 <vertex x="0" y="55.88"/>
 </polygon>
+<wire x1="68.58" y1="16.51" x2="76.2" y2="11.43" width="0" layer="19" extent="1-1"/>
+<wire x1="45.72" y1="15.24" x2="68.58" y2="16.51" width="0" layer="19" extent="1-1"/>
+<wire x1="45.72" y1="10.16" x2="45.72" y2="15.24" width="0" layer="19" extent="1-1"/>
+<wire x1="33.02" y1="10.16" x2="45.72" y2="10.16" width="0" layer="19" extent="1-1"/>
+<wire x1="10.16" y1="44.45" x2="33.02" y2="10.16" width="0" layer="19" extent="1-1"/>
+<wire x1="8.37" y1="51.23" x2="10.16" y2="44.45" width="0" layer="19" extent="1-1"/>
 </signal>
 <signal name="5V">
@@
 <wire x1="62.23" y1="24.13" x2="68.58" y2="24.13" width="0.4064" layer="1"/>
 </signal>
-<signal name="N$8">
-<contactref element="R5" pad="1"/>
-<contactref element="DISPLAY" pad="3"/>
-<wire x1="55.88" y1="36.83" x2="59.69" y2="36.83" width="0.4064" layer="1"/>
-</signal>
 </signals>

Commit message: board changes & template init finished
Other:
- board text added: "Internet of Plants"
- board text added: "Prototype 2"
Changed lines of the file:
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@@
 <text x="4.445" y="9.525" size="0.6096" layer="25">+12V</text>
 <text x="5.08" y="17.78" size="0.6096" layer="25">GND</text>
-<text x="81.28" y="52.07" size="0.6096" layer="26" rot="MR0">2017 Bilal Mahmoud</text>
+<text x="84.455" y="52.07" size="1.27" layer="22" font="vector" rot="MR0">2017 Bilal Mahmoud</text>
 <text x="58.42" y="7.62" size="0.8128" layer="26" rot="MR0">"Nothing is work unless you'd rather be doing something else" - George Halas</text>
 <wire x1="41.91" y1="8.89" x2="44.45" y2="11.43" width="0.4064" layer="21" curve="-90"/>
@@
 <wire x1="27.94" y1="43.18" x2="27.94" y2="45.72" width="0.4064" layer="21"/>
 <wire x1="7.62" y1="43.18" x2="7.62" y2="45.72" width="0.4064" layer="21"/>
+<text x="84.455" y="45.72" size="1.016" layer="22" rot="MR0">Prototype 2</text>
+<text x="84.455" y="46.99" size="1.016" layer="22" rot="MR0">Internet of Plants</text>
 </plain>
 <attributes>
@@
 <contactref element="DISPLAY" pad="3"/>
 <contactref element="DISPLAY" pad="5"/>
-<wire x1="73.66" y1="50.8" x2="80.01" y2="50.8" width="0" layer="19" extent="1-1"/>
-<wire x1="67.31" y1="50.8" x2="73.66" y2="50.8" width="0" layer="19" extent="1-1"/>
-<wire x1="59.69" y1="39.37" x2="67.31" y2="50.8" width="0" layer="19" extent="1-1"/>
-<wire x1="59.69" y1="36.83" x2="59.69" y2="39.37" width="0" layer="19" extent="1-1"/>
-<wire x1="59.69" y1="34.29" x2="59.69" y2="36.83" width="0" layer="19" extent="1-1"/>
-<wire x1="68.58" y1="13.97" x2="59.69" y2="34.29" width="0" layer="19" extent="1-1"/>
-<wire x1="76.2" y1="8.89" x2="68.58" y2="13.97" width="0" layer="19" extent="1-1"/>
-<wire x1="76.2" y1="6.35" x2="76.2" y2="8.89" width="0" layer="19" extent="1-1"/>
-<wire x1="76.2" y1="3.81" x2="76.2" y2="6.35" width="0" layer="19" extent="1-1"/>
-<wire x1="82.55" y1="16.51" x2="76.2" y2="8.89" width="0" layer="19" extent="1-1"/>
-<wire x1="53.34" y1="10.16" x2="68.58" y2="13.97" width="0" layer="19" extent="1-1"/>
-<wire x1="25.4" y1="2.54" x2="53.34" y2="10.16" width="0" layer="19" extent="1-1"/>
-<wire x1="15.24" y1="2.54" x2="25.4" y2="2.54" width="0" layer="19" extent="1-1"/>
-<wire x1="5.08" y1="15.67" x2="15.24" y2="2.54" width="0" layer="19" extent="1-1"/>
-<wire x1="12.7" y1="19.05" x2="5.08" y2="15.67" width="0" layer="19" extent="1-1"/>
-<wire x1="12.7" y1="21.59" x2="12.7" y2="19.05" width="0" layer="19" extent="1-1"/>
-<wire x1="12.7" y1="44.45" x2="12.7" y2="21.59" width="0" layer="19" extent="1-1"/>
-<wire x1="18.5166" y1="51.2318" x2="12.7" y2="44.45" width="0" layer="19" extent="1-1"/>
 </signal>
 <signal name="VCC">
@@
 <vertex x="0" y="55.88"/>
 </polygon>
-<wire x1="68.58" y1="16.51" x2="76.2" y2="11.43" width="0" layer="19" extent="1-1"/>
-<wire x1="45.72" y1="15.24" x2="68.58" y2="16.51" width="0" layer="19" extent="1-1"/>
-<wire x1="45.72" y1="10.16" x2="45.72" y2="15.24" width="0" layer="19" extent="1-1"/>
-<wire x1="33.02" y1="10.16" x2="45.72" y2="10.16" width="0" layer="19" extent="1-1"/>
-<wire x1="10.16" y1="44.45" x2="33.02" y2="10.16" width="0" layer="19" extent="1-1"/>
-<wire x1="8.37" y1="51.23" x2="10.16" y2="44.45" width="0" layer="19" extent="1-1"/>
 </signal>
 <signal name="5V">
