File: pcbs/rpi-hat-exp/main.sch (EAGLE design)
At the start: 15 parts, among them IC1 MCP23017, IC2 L293D, J2 1X2-3.5MM, J3 1X2-3.5MM, U1 MCP3002

Commit message: I changed 'some' stuff
Parts:
- removed LED1: RGBLED_CA-5MM, adafruit:RGBLED_CA-5MM
- removed R1: 220, adafruit:R-US_0204/7
- removed R2: 330, adafruit:R-US_0204/7
- added LED2: WS2812BTH, adafruit:WS2812BTH
Connections:
- removed net GPIO13M: LED1.RED, R1.1, R2.2
- new net GPIO18: JP2.GPIO18, LED2.DI
- net GND: now also LED2.GND; no longer LED1.VCC, R2.1
- net GPIO05: no longer LED1.BLUE
- net GPIO06: no longer LED1.GREEN
- net GPIO13: no longer R1.2
- net VCC: now also LED2.VDD
Changed lines of the file:
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@@
 <part name="GND21" library="supply1" deviceset="GND" device=""/>
 <part name="GND22" library="supply1" deviceset="GND" device=""/>
-<part name="LED1" library="adafruit" deviceset="RGBLED_CA" device="-5MM"/>
-<part name="GND23" library="supply1" deviceset="GND" device=""/>
-<part name="R1" library="adafruit" deviceset="R-US_" device="0204/7" value="220"/>
-<part name="R2" library="adafruit" deviceset="R-US_" device="0204/7" value="330"/>
-<part name="GND1" library="supply1" deviceset="GND" device=""/>
+<part name="LED2" library="adafruit" deviceset="WS2812B" device="TH"/>
+<part name="P+1" library="supply1" deviceset="VCC" device=""/>
+<part name="GND11" library="supply1" deviceset="GND" device=""/>
 </parts>
 <sheets>
@@
 <instance part="GND21" gate="1" x="99.06" y="86.36" rot="R90"/>
 <instance part="GND22" gate="1" x="99.06" y="96.52" rot="R90"/>
-<instance part="LED1" gate="G$1" x="63.5" y="22.86" rot="R90"/>
-<instance part="GND23" gate="1" x="63.5" y="10.16"/>
-<instance part="R1" gate="G$1" x="86.36" y="30.48" rot="R90"/>
-<instance part="R2" gate="G$1" x="86.36" y="15.24" rot="R90"/>
-<instance part="GND1" gate="1" x="86.36" y="5.08"/>
+<instance part="LED2" gate="G$1" x="33.02" y="0"/>
+<instance part="P+1" gate="VCC" x="38.1" y="17.78"/>
+<instance part="GND11" gate="1" x="33.02" y="-12.7"/>
 </instances>
 <busses>
@@
 </segment>
 <segment>
-<pinref part="LED1" gate="G$1" pin="VCC"/>
-<pinref part="GND23" gate="1" pin="GND"/>
-</segment>
-<segment>
-<pinref part="R2" gate="G$1" pin="1"/>
-<pinref part="GND1" gate="1" pin="GND"/>
-<wire x1="86.36" y1="7.62" x2="86.36" y2="10.16" width="0.1524" layer="91"/>
+<pinref part="LED2" gate="G$1" pin="GND"/>
+<pinref part="GND11" gate="1" pin="GND"/>
 </segment>
 </net>
@@
 <pinref part="JP2" gate="A" pin="3V3@1"/>
 <pinref part="P+11" gate="VCC" pin="VCC"/>
+</segment>
+<segment>
+<pinref part="LED2" gate="G$1" pin="VDD"/>
+<pinref part="P+1" gate="VCC" pin="VCC"/>
 </segment>
 </net>
@@
 <label x="53.34" y="60.96" size="1.778" layer="95" rot="R180" xref="yes"/>
 </segment>
-<segment>
-<wire x1="86.36" y1="38.1" x2="86.36" y2="35.56" width="0.1524" layer="91"/>
-<pinref part="R1" gate="G$1" pin="2"/>
-<label x="86.36" y="38.1" size="1.778" layer="95" rot="R90" xref="yes"/>
-</segment>
 </net>
 <net name="N$1" class="0">
@@
 <label x="66.04" y="63.5" size="1.778" layer="95" rot="R180" xref="yes"/>
 </segment>
-<segment>
-<pinref part="LED1" gate="G$1" pin="GREEN"/>
-<wire x1="63.5" y1="30.48" x2="63.5" y2="33.02" width="0.1524" layer="91"/>
-<label x="63.5" y="33.02" size="1.778" layer="95" rot="R90" xref="yes"/>
-</segment>
 </net>
 <net name="GPIO05" class="0">
@@
 <label x="53.34" y="66.04" size="1.778" layer="95" rot="R180" xref="yes"/>
 </segment>
-<segment>
-<pinref part="LED1" gate="G$1" pin="BLUE"/>
-<wire x1="58.42" y1="30.48" x2="58.42" y2="33.02" width="0.1524" layer="91"/>
-<label x="58.42" y="33.02" size="1.778" layer="95" rot="R90" xref="yes"/>
-</segment>
-</net>
-<net name="GPIO13M" class="0">
-<segment>
-<pinref part="LED1" gate="G$1" pin="RED"/>
-<wire x1="68.58" y1="30.48" x2="68.58" y2="33.02" width="0.1524" layer="91"/>
-<label x="68.58" y="33.02" size="1.778" layer="95" rot="R90" xref="yes"/>
-</segment>
-<segment>
-<pinref part="R1" gate="G$1" pin="1"/>
-<pinref part="R2" gate="G$1" pin="2"/>
-<wire x1="86.36" y1="25.4" x2="86.36" y2="22.86" width="0.1524" layer="91"/>
-<wire x1="86.36" y1="22.86" x2="86.36" y2="20.32" width="0.1524" layer="91"/>
-<wire x1="86.36" y1="22.86" x2="93.98" y2="22.86" width="0.1524" layer="91"/>
-<junction x="86.36" y="22.86"/>
-<label x="93.98" y="22.86" size="1.778" layer="95" xref="yes"/>
-</segment>
-</net>
+</net>
+<net name="GPIO18" class="0">
+<segment>
+<pinref part="JP2" gate="A" pin="GPIO18"/>
+<wire x1="96.52" y1="88.9" x2="109.22" y2="88.9" width="0.1524" layer="91"/>
+<label x="109.22" y="88.9" size="1.778" layer="95" xref="yes"/>
+</segment>
+<segment>
+<pinref part="LED2" gate="G$1" pin="DI"/>
+<wire x1="20.32" y1="-2.54" x2="15.24" y2="-2.54" width="0.1524" layer="91"/>
+<label x="15.24" y="-2.54" size="1.778" layer="95" rot="R180" xref="yes"/>
+</segment>
+</net>
